File: ATF2FT232HQ/ATF2FT232HQ.kicad_pcb (KiCad board)
At the start: 2 copper layers, 83.8 x 44.4 mm, 23 parts, among them J1 USB, J2 JTAG, SW1 Vcc, SW2 Vpp, U1 ATF15xx, U2 MAX662A

Commit message: Fix switch footprint.
Parts:
- C1, C2, C3, C4: moved to F.Cu
- SW1, SW2: footprint T-Pau:SW_Apem_SS-25136-NH -> T-Pau:SS2513
- moved SW2 6.29 mm to (145.5, 56.0)
- moved SW1 6.25 mm to (145.5, 74.8)
- moved C1 0.53 mm to (99.2, 85.1)
- moved C3 0.33 mm to (115.2, 71.2)
Routing:
- net +5V: track 32.1 -> 34.9 mm
- net +3V3: track 13.9 -> 16.6 mm
- net Net-(SW2-A): track 17.6 -> 20.0 mm
- net VCC: track 108.5 -> 109.0 mm
Other:
- board text added: "Vcc"
- board text added: "Vpp"
