File: ATF2FT232HQ/ATF2FT232HQ.kicad_sch (KiCad schematic)
At the start: 23 parts, among them J1 USB, J2 JTAG, SW1 Vcc, SW2 Vpp, U1 ATF15xx, U2 MAX662A

Commit message: Fix switch footprint.
Parts:
- SW1, SW2: footprint T-Pau:SW_Apem_SS-25136-NH -> T-Pau:SS2513
Changed lines of the file:
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@@
 			)
 		)
-		(property "Footprint" "T-Pau:SW_Apem_SS-25136-NH"
+		(property "Footprint" "T-Pau:SS2513"
 			(at 46.99 104.14 0)
 			(effects
@@
 			)
 		)
-		(property "Footprint" "T-Pau:SW_Apem_SS-25136-NH"
+		(property "Footprint" "T-Pau:SS2513"
 			(at 106.68 58.42 0)
 			(effects
